File: hardware/ss_pcb_rev1_0/ss_pcb_rev1_0.kicad_pcb (KiCad board)
At the start: 2 copper layers, 50 x 60 mm, 11 parts, among them J3 Micro_SD_Card_Module, SW1 SW_Push, SW2 SW_Push, SW3 SW_Push, SW4 SW_Push, U1 esp32_devkit_WROOM-32, U2 LCD_Module_ST7735

Commit message: updates rev_0 hw design files.
Routing:
- net LCD_GND: track 0.00 -> 146.3 mm, vias 0 -> 1
- net LCD_VCC: track 0.00 -> 121.8 mm
- net SW_BACK: track 0.00 -> 44.8 mm
- net SW_OK: track 0.00 -> 34.6 mm
- net SW_DOWN: track 0.00 -> 26.6 mm
- net LCD_BL: track 0.00 -> 26.5 mm
- net SW_UP: track 0.00 -> 20.4 mm
- net LCD_SPI_CS: track 25.7 -> 40.7 mm
- net LCD_SPI_CLK: track 33.0 -> 38.7 mm, vias 0 -> 1
- net LCD_DC: track 34.8 -> 32.5 mm
- net LCD_RESET: track 30.9 -> 28.9 mm
- net LCD_SPI_MOSI: track 28.1 -> 28.8 mm, vias 0 -> 1
